File: hardware/redunDCv1/redunDCv1.kicad_pcb (KiCad board)
At the start: 2 copper layers, 71 parts, among them J1 PS1_ALARM, J11 OUT1, J12 OUT2, J13 OUT3, J14 OUT4, J15 OUT5, J16 OUT6, J17 OUT7, J18 OUT8, J2 PS1_PWR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

Commit message: some routing tests...
Parts:
- moved H1 272.8 mm to (260.4, 32.6)
- moved H2 272.8 mm to (260.4, 40.6)
- moved H3 272.8 mm to (268.3, 32.6)
- moved H4 272.8 mm to (268.3, 40.6)
- moved H5 272.8 mm to (276.2, 32.6)
- moved H6 272.8 mm to (276.2, 40.6)
- moved J6 81.3 mm to (182.9, 31.5), turned to 0 degrees
- moved D13 56.1 mm to (206.1, 55.2)
- moved D16 56.1 mm to (233.7, 63.0)
- moved D6 56.1 mm to (103.5, 54.5)
- moved C1 56.1 mm to (46.4, 70.4)
- moved C2 56.1 mm to (73.0, 70.6)
- moved C3 56.1 mm to (99.3, 69.1)
- moved C4 56.1 mm to (130.0, 70.7)
- moved C5 56.1 mm to (150.2, 70.6)
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Routing:
- net GND: track 0.00 -> 154.4 mm, vias 0 -> 1
- net /PS1_AC-OK: track 0.00 -> 99.9 mm
- net /PS1_BAT-LOW: track 0.00 -> 96.9 mm, vias 0 -> 2
- net +12V: track 0.00 -> 81.2 mm
- net /PS2_V+: track 0.00 -> 71.8 mm
- net /PS1_V+: track 0.00 -> 46.3 mm
- net /PS2_BAT-: track 0.00 -> 38.4 mm
- net /PS1_BAT-: track 0.00 -> 38.3 mm
- net /PS2_BAT-LOW: track 0.00 -> 32.1 mm, vias 0 -> 1
- net /PS2_AC-OK: track 0.00 -> 24.5 mm, vias 0 -> 2
- net /PS2_BAT+: track 0.00 -> 16.9 mm
- net /PS1_BAT+: track 0.00 -> 16.8 mm
- net Net-(R6-Pad2): track 0.00 -> 15.5 mm, vias 0 -> 2
- net Net-(LS1-Pad2): track 0.00 -> 14.9 mm
- net Net-(D17-Pad1): track 0.00 -> 8.00 mm
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Other:
- net class High-Power added: clearance 0.2, trace_width 3, via_dia 3.2, via_drill 0.6
- net class Power added: clearance 0.2, trace_width 0.5, via_dia 0.7, via_drill 0.5
