File: hardware/redunDCv1/mcu.sch (KiCad schematic (older format))
At the start: 20 parts

Commit message: added symbols for isolators
Parts:
- added C? (x3): 100nF, symbol Device:C_Small
- added C?: 1µF, symbol Device:CP_Small
- added R? (x2): 3k3, symbol Device:R_Small
- added R? (x2): 6k8, symbol Device:R_Small
- added U?: ATtiny102-SS, Package_SO:SOIC-8_3.9x4.9mm_P1.27mm, symbol MCU_Microchip_ATtiny:ATtiny102-SS
- added U?: Si8621, Package_SO:SOIC-8_3.9x4.9mm_P1.27mm, symbol redundc:Si8621
- added U?: TME0505S, symbol redundc:TME0505S
Connections:
- net labels added: +5VL, GND
- wire segments 73 -> 119
- no-connect marks 1 -> 3

Commit message: schemativ almost done
Parts:
- removed U?: ATtiny102-SS, Package_SO:SOIC-8_3.9x4.9mm_P1.27mm, symbol MCU_Microchip_ATtiny:ATtiny102-SS
- added J?: ICSP, symbol Connector_Generic:Conn_02x03_Odd_Even
- added Q? (x4): BS170F, Package_TO_SOT_SMD:SOT-23, symbol Transistor_FET:BS170F
- added R? (x4): 100R, symbol Device:R_Small
- added R? (x2): 10k, symbol Device:R_Small
- added SW?: Reset B, symbol Switch:SW_Push
- added U?: ATtiny1634-SU, Package_SO:SOIC-20W_7.5x12.8mm_P1.27mm, symbol MCU_Microchip_ATtiny:ATtiny1634-SU
- SW?: value Reset -> Reset A
Connections:
- net labels added: MISO_B, MOSI_B, PS1_AC-OK_SENSE, PS1_BAT-LOW_SENSE, PS2_AC-OK_SENSE, PS2_BAT-LOW_SENSE, RXD_A, RXD_B, SCK_B, TXD_A, TXD_B, VS1_SENSE, VS2_SENSE
- net labels removed: PS1_AC_OK
- wire segments 119 -> 162
- no-connect marks 3 -> 7
Other:
- moved on the sheet: C?, D?, J?, L?, R?, SW?, U?, Y?
